Commit message: Baselink frame in URDF for map navi |  Fixing the lidar params in cost map common in go1_navigation

File: go1_description/urdf/go1_robotis.urdf (robot description, URDF)
Before this commit: robot go1, 56 links, 55 joints
Links:
- added link base_link
Joints:
- added joint base_link_joint: type fixed, parent base, child base_link, origin xyz=0 0 0 rpy=0 0 0
