Commit message: PointCloud2 to LaserScan | SLAM  are working
The conversion from point cloud to scan information is working now. The frame name and topic are updated. Also for the HECTOR Slam, a extra frame is added in the urdf of the robot.

File: go1_description/urdf/go1.urdf (robot description, URDF)
Before this commit: robot go1, 38 links, 37 joints
Links:
- added link base_footprint
Joints:
- added joint base_footprint_joint: type fixed, parent base, child base_footprint, origin xyz=0 0 0 rpy=0 0 0

Commit message: Making N13 same as N14. No need of two branches

File: go1_description/urdf/go1.urdf (robot description, URDF)
Before this commit: robot go1, 39 links, 38 joints
Links:
- removed link base_footprint
Joints:
- removed joint base_footprint_joint

File: go1_description/urdf/go1_robotis.urdf (robot description, URDF)
Before this commit: robot go1, 55 links, 54 joints
Links:
- added link base_footprint
- added link base_link
Joints:
- added joint base_footprint_joint: type fixed, parent base, child base_footprint, origin xyz=0 0 0 rpy=0 0 0
- added joint base_link_joint: type fixed, parent base, child base_link, origin xyz=0 0 0 rpy=0 0 0
